Commit message: update xacro macro with new rigid body model

File: urdf/macro_definitions.urdf.xacro (robot description, xacro)
@@ -7,15 +7,15 @@
     <color rgba="1 1 1 1"/>
   </material>
-  <material name="red">
-    <color rgba="1 0 0 1"/>
+  <material name="green">
+    <color rgba="0.2 1 0.2 0.8"/>
   </material>
   <xacro:property name="PI" value="3.1415" />
   <xacro:macro name="ball-joint" params="id parent child">
-    <!--creates a ball joint, called from the PCC macro..-->
+    <!--creates a (pseudo) ball joint, called from the PCC macro..-->
     <joint name="${id}-ball-joint_x_joint" type="revolute">
       <parent link="${parent}"/>
       <child link="${id}-ball-joint_link_0"/>
       <axis xyz="1 0 0"/>
-      <limit lower="${-PI/4}" upper="${PI/4}" effort="1000" velocity="1000"/>
+      <limit lower="${-PI/2}" upper="${PI/2}" effort="1000" velocity="1000"/>
     </joint>
     <link name="${id}-ball-joint_link_0">
@@ -26,5 +26,5 @@
       <child link="${id}-ball-joint_link_1"/>
       <axis xyz="0 1 0"/>
-      <limit lower="${-PI/4}" upper="${PI/4}" effort="1000" velocity="1000"/>
+      <limit lower="${-PI/2}" upper="${PI/2}" effort="1000" velocity="1000"/>
     </joint>
     <link name="${id}-ball-joint_link_1">
@@ -41,16 +41,6 @@
       <child link="${child}"/>
       <axis xyz="0 0 1"/>
-      <limit lower="${-PI/4}" upper="${PI/4}" effort="1000" velocity="1000"/>
+      <limit lower="${-PI/2}" upper="${PI/2}" effort="1000" velocity="1000"/>
     </joint>
-  </xacro:macro>
-  <xacro:macro name="rod" params="length direction=1">
-    <!--creates a visual of a rod.-->
-    <visual>
-      <geometry>
-        <cylinder radius="${length/50}" length="${length/2}"/>
-      </geometry>
-      <material name="white"/>
-      <origin xyz="0 0 ${direction*length/4}"/>
-    </visual>
   </xacro:macro>
   <xacro:macro name="default_inertial">
@@ -61,10 +51,9 @@
     </inertial>
   </xacro:macro>
-  <xacro:macro name="PCC" params="id parent child length mass">
+  <xacro:macro name="PCC" params="id parent child length mass radius:=0.02">
     <!--creates a PCC piece-->
-    <xacro:ball-joint id="${id}-base" parent="${parent}" child="${id}-a"/>
+    <xacro:ball-joint id="${id}-ball" parent="${parent}" child="${id}-a"/>
     <link name="${id}-a">
       <xacro:default_inertial/>
-      <xacro:rod length="${length}"/>
     </link>
     <joint name="${id}-a-b_joint" type="prismatic">
@@ -78,7 +67,8 @@
       <visual>
         <geometry>
-          <box size="${length/4} ${length/4} ${length/4}"/>
+          <cylinder length="${length}" radius="${radius}"/>
         </geometry>
-        <material name="red"/>
+        <!-- <origin xyz="0 0 ${length/2}"/> -->
+        <material name="green"/>
       </visual>
       <inertial>
@@ -87,20 +77,11 @@
       </inertial>
     </link>
-    <xacro:ball-joint id="${id}-middle" parent="${id}-b" child="${id}-c"/>
-    <link name="${id}-c">
-      <xacro:default_inertial/>
-    </link>
-    <joint name="${id}-c-d_joint" type="prismatic">
-      <parent link="${id}-c"/>
-      <child link="${id}-d"/>
+    <joint name="${id}-b-${child}_joint" type="prismatic">
+      <parent link="${id}-b"/>
+      <child link="${child}"/>
       <axis xyz="0 0 -1"/>
       <origin xyz="0 0 ${length/2}"/>
       <limit lower="0" upper="${length/2}" effort="1000" velocity="1000"/>
     </joint>
-    <link name="${id}-d">
-      <xacro:default_inertial/>
-      <xacro:rod length="${length}" direction="-1"/>
-    </link>
-    <xacro:ball-joint id="${id}-tip" parent="${id}-d" child="${child}"/>
   </xacro:macro>
   <xacro:macro name="empty_link" params="name">

Commit message: set cylinder rotational inertia

File: urdf/macro_definitions.urdf.xacro (robot description, xacro)
@@ -4,7 +4,4 @@
 -->
 <robot xmlns:xacro="http://www.ros.org/wiki/xacro" name="robot">
-  <material name="white">
-    <color rgba="1 1 1 1"/>
-  </material>
   <material name="green">
     <color rgba="0.2 1 0.2 0.8"/>
@@ -30,11 +27,5 @@
     <link name="${id}-ball-joint_link_1">
       <xacro:default_inertial/>
-      <visual>
-        <geometry>
-          <box size="${length/10} ${length/10} ${length/10}"/>
-        </geometry>
-        <material name="white"/>
-      </visual>
-    </link>
+   </link>
     <joint name="${id}-ball-joint_z_joint" type="revolute">
       <parent link="${id}-ball-joint_link_1"/>
@@ -74,5 +65,6 @@
       <inertial>
         <mass value="${mass}"/>
-        <inertia ixx="0.0001" ixy="0.000" ixz="0.000" iyy="0.0001" iyz="0.000" izz="0.0001"/>
+        <!-- moment of inertia for a cylinder with radius and length -->
+        <inertia ixx="${mass * (3*radius**2 + length**2) / 12.}" ixy="0.000" ixz="0.000" iyy="${mass * (3*radius**2 + length**2) / 12.}" iyz="0.000" izz="${mass * radius*radius / 2.}"/>
       </inertial>
     </link>

Commit message: add mark to URDF marking first chamber, can set angle of arm

File: urdf/macro_definitions.urdf.xacro (robot description, xacro)
@@ -6,4 +6,7 @@
   <material name="green">
     <color rgba="0.2 1 0.2 0.8"/>
+  </material>
+  <material name="white">
+    <color rgba="0.5 0.5 0.5 1"/>
   </material>
   <xacro:property name="PI" value="3.1415" />
@@ -63,4 +66,12 @@
         <material name="green"/>
       </visual>
+      <visual>
+        <!-- this marks the +x direction (i.e. the direction where the first chamber should be) -->
+        <geometry>
+          <box size="${radius/5.} ${radius/5.} ${radius/5.}"/>
+        </geometry>
+        <origin xyz="${radius} 0 0"/>
+        <material name="white"/>
+      </visual>
       <inertial>
         <mass value="${mass}"/>

Commit message: add simple ROS visualizer

File: urdf/macro_definitions.urdf.xacro (robot description, xacro)
@@ -93,3 +93,10 @@
     </link>
   </xacro:macro>
+  <xacro:macro name="rigid_rotation" params="rotX rotY rotZ parent child">
+    <joint name="${parent}_${child}_joint" type="fixed">
+      <parent link="${parent}"/>
+      <child link="${child}"/>
+      <origin rpy="${rotX} ${rotY} ${rotZ}"/>
+    </joint>
+  </xacro:macro>
 </robot>

Commit message: create new joints required to match CoM

File: urdf/macro_definitions.urdf.xacro (robot description, xacro)
@@ -60,4 +60,11 @@
     </joint>
     <link name="${id}-b">
+      <xacro:default_inertial/>
+    </link>
+    <!-- These links branch out into the XY plane. The mass can move around the plane to match the CoM of the actual PCC model -->
+    <link name="${id}-branch-a">
+      <xacro:default_inertial/>
+    </link>
+    <link name="${id}-branch-b">
       <visual>
         <geometry>
@@ -81,4 +88,17 @@
       </inertial>
     </link>
+    <!-- the next two joints are prismatic joints to move the mass on a plane to match CoM position -->
+    <joint name="${id}-b-branch-a_joint" type="prismatic">
+      <parent link="${id}-b"/>
+      <child link="${id}-branch-a"/>
+      <axis xyz="1 0 0"/>
+      <limit lower="-1" upper="1" effort="1000" velocity="1000"/>
+    </joint>
+    <joint name="${id}-branch-a-branch-b_joint" type="prismatic">
+      <parent link="${id}-branch-a"/>
+      <child link="${id}-branch-b"/>
+      <axis xyz="0 1 0"/>
+      <limit lower="-1" upper="1" effort="1000" velocity="1000"/>
+    </joint>
     <joint name="${id}-b-${child}_joint" type="prismatic">
       <parent link="${id}-b"/>

Commit message: Xacro fixed

File: urdf/macro_definitions.urdf.xacro (robot description, xacro)
@@ -60,11 +60,4 @@
     </joint>
     <link name="${id}-b">
-      <xacro:default_inertial/>
-    </link>
-    <!-- These links branch out into the XY plane. The mass can move around the plane to match the CoM of the actual PCC model -->
-    <link name="${id}-branch-a">
-      <xacro:default_inertial/>
-    </link>
-    <link name="${id}-branch-b">
       <visual>
         <geometry>
@@ -88,17 +81,4 @@
       </inertial>
     </link>
-    <!-- the next two joints are prismatic joints to move the mass on a plane to match CoM position -->
-    <joint name="${id}-b-branch-a_joint" type="prismatic">
-      <parent link="${id}-b"/>
-      <child link="${id}-branch-a"/>
-      <axis xyz="1 0 0"/>
-      <limit lower="-1" upper="1" effort="1000" velocity="1000"/>
-    </joint>
-    <joint name="${id}-branch-a-branch-b_joint" type="prismatic">
-      <parent link="${id}-branch-a"/>
-      <child link="${id}-branch-b"/>
-      <axis xyz="0 1 0"/>
-      <limit lower="-1" upper="1" effort="1000" velocity="1000"/>
-    </joint>
     <joint name="${id}-b-${child}_joint" type="prismatic">
       <parent link="${id}-b"/>
