Commit message: Update example_prismatic.urdf

File: urdf/example_prismatic.urdf (robot description, URDF)
Before this commit: robot 2segment, 53 links, 52 joints
Links:
- link prism_base_link: geometry visual cylinder length=0.024 radius=0.1
- link prism_lower_link: geometry visual cylinder length=0.15 radius=0.1

Commit message: Update example_prismatic.urdf

File: urdf/example_prismatic.urdf (robot description, URDF)
Before this commit: robot 2segment, 53 links, 52 joints
Links:
- link prism_base_link: geometry visual cylinder length=0.05 radius=0.05
- link prism_lower_link: geometry visual cylinder length=0.10 radius=0.05

Commit message: Update example_prismatic.urdf

File: urdf/example_prismatic.urdf (robot description, URDF)
Before this commit: robot 2segment, 53 links, 52 joints
Joints:
- joint prism_joint: limit lower=0 upper=0.08 effort=1000 velocity=1000 -> lower=0.08 upper=0 effort=1000 velocity=1000

Commit message: Update example_prismatic.urdf

File: urdf/example_prismatic.urdf (robot description, URDF)
Before this commit: robot 2segment, 53 links, 52 joints
Joints:
- joint prism_joint: axis 0 0 -1 -> 0 0 1; limit lower=0.08 upper=0 effort=1000 velocity=1000 -> lower=0 upper=0.08 effort=1000 velocity=1000

Commit message: Update example_prismatic.urdf

File: urdf/example_prismatic.urdf (robot description, URDF)
Before this commit: robot 2segment, 53 links, 52 joints
Links:
- link prism_base_link: geometry visual cylinder length=0.01 radius=0.05

Commit message: Update example_prismatic.urdf

File: urdf/example_prismatic.urdf (robot description, URDF)
Before this commit: robot 2segment, 53 links, 52 joints
Links:
- link prism_base_link: geometry visual cylinder length=0.1 radius=0.03

Commit message: Update example_prismatic.urdf

File: urdf/example_prismatic.urdf (robot description, URDF)
Before this commit: robot 2segment, 53 links, 52 joints
Links:
- link prism_base_link: geometry visual cylinder length=0.1 radius=0.01
- link prism_lower_link: geometry visual cylinder length=0.10 radius=0.009

Commit message: Update example_prismatic.urdf

File: urdf/example_prismatic.urdf (robot description, URDF)
Before this commit: robot 2segment, 53 links, 52 joints
Links:
- link prism_base_link: geometry visual cylinder length=0.01 radius=0.03
- link prism_lower_link: geometry visual cylinder length=0.15 radius=0.05

Commit message: Update example_prismatic.urdf

File: urdf/example_prismatic.urdf (robot description, URDF)
Before this commit: robot 2segment, 53 links, 52 joints
Links:
- link prism_lower_link: geometry visual cylinder length=0.15 radius=0.04

Commit message: Update example_prismatic.urdf

File: urdf/example_prismatic.urdf (robot description, URDF)
Before this commit: robot 2segment, 53 links, 52 joints
Links:
- link prism_base_link: geometry visual cylinder length=0.15 radius=0.04
- link prism_lower_link: geometry visual cylinder length=0.15 radius=0.02

Commit message: Update example_prismatic.urdf

File: urdf/example_prismatic.urdf (robot description, URDF)
Before this commit: robot 2segment, 53 links, 52 joints
Links:
- link prism_base_link: geometry visual cylinder length=0.15 radius=0.02
- link prism_lower_link: geometry visual cylinder length=0.15 radius=0.03
